Commit message: fixed humanoid movement

File: data/humanoid.urdf (robot description, URDF)
Before this commit: robot , 34 links, 33 joints
Joints:
- joint abdomen_x: type continuous -> fixed
- joint abdomen_y: type continuous -> fixed
- joint abdomen_z: type continuous -> fixed
- joint left_hip_x: type continuous -> fixed
- joint right_hip_x: type continuous -> fixed

Commit message: modified humanoid.urdf

File: data/humanoid.urdf (robot description, URDF)
Before this commit: robot , 34 links, 33 joints
Links:
- link left_foot: geometry collision box size=0.05400 0.05400 0.21095; collision box size=0.05400 0.05400 0.21095
- link left_lower_arm: geometry collision box size=0.06200 0.06200 0.27713; collision box size=0.08000 0.08000 0.08000
- link left_shin: geometry collision box size=0.09800 0.09800 0.30000
- link left_thigh: geometry collision box size=0.12000 0.12000 0.34015
- link left_upper_arm: geometry collision box size=0.08000 0.08000 0.27713
- link link1_11: mass 0.00000 -> 0.00001
- link link1_13: mass 0.00000 -> 0.00001
- link link1_14: mass 0.00000 -> 0.00001
- link link1_16: mass 0.00000 -> 0.00001
- link link1_17: mass 0.00000 -> 0.00001
- link link1_18: mass 0.00000 -> 0.00001
- link link1_2: mass 0.00000 -> 0.00001
- link link1_20: mass 0.00000 -> 0.00001
- link link1_22: mass 0.00000 -> 0.00001
- link link1_23: mass 0.00000 -> 0.00001
- link link1_25: mass 0.00000 -> 0.00001
- link link1_26: mass 0.00000 -> 0.00001
- link link1_28: mass 0.00000 -> 0.00001
- link link1_3: mass 0.00000 -> 0.00001
- link link1_30: mass 0.00000 -> 0.00001
- link link1_31: mass 0.00000 -> 0.00001
- link link1_33: mass 0.00000 -> 0.00001
- link link1_5: mass 0.00000 -> 0.00001
- link link1_7: mass 0.00000 -> 0.00001
- link link1_8: mass 0.00000 -> 0.00001
- link link1_9: mass 0.00000 -> 0.00001
- link lwaist: geometry collision box size=0.12000 0.12000 0.12000
- link pelvis: geometry collision box size=0.18000 0.18000 0.14000
- link right_foot: geometry collision box size=0.05400 0.05400 0.21095; collision box size=0.05400 0.05400 0.21095
- link right_lower_arm: geometry collision box size=0.06200 0.06200 0.27713; collision box size=0.08000 0.08000 0.08000
- link right_shin: geometry collision box size=0.09800 0.09800 0.30000
- link right_thigh: geometry collision box size=0.12000 0.12000 0.34015
- link right_upper_arm: geometry collision box size=0.08000 0.08000 0.27713
- link torso: geometry collision box size=0.12000 0.12000 0.12000; collision box size=0.14000 0.14000 0.14000
Joints:
- joint abdomen_y: limit (none) -> lower=-0.5 upper=0.5 effort=100.0 velocity=10.0; type fixed -> revolute
- joint left_ankle_x: type continuous -> fixed
- joint left_ankle_y: limit (none) -> lower=-0.7 upper=0.7 effort=100.0 velocity=10.0; type continuous -> revolute
- joint left_elbow: axis 0.00000 -1.00000 -1.00000 -> 0.00000 1.00000 0.00000; limit (none) -> lower=0.0 upper=2.5 effort=100.0 velocity=10.0; type continuous -> revolute
- joint left_hip_x: limit (none) -> lower=-0.8 upper=0.8 effort=100.0 velocity=10.0; type fixed -> revolute
- joint left_hip_y: type continuous -> fixed
- joint left_hip_z: limit (none) -> lower=-1.5 upper=0.5 effort=100.0 velocity=10.0; type continuous -> revolute
- joint left_knee: limit (none) -> lower=0.0 upper=2.0 effort=100.0 velocity=10.0; type continuous -> revolute
- joint left_shoulder1: axis 2.00000 -1.00000 1.00000 -> 0.00000 1.00000 0.00000; limit (none) -> lower=-2.0 upper=2.0 effort=100.0 velocity=10.0; type continuous -> revolute
- joint left_shoulder2: axis 0.00000 1.00000 1.00000 -> 1.00000 0.00000 0.00000; limit (none) -> lower=-1.0 upper=1.0 effort=100.0 velocity=10.0; type continuous -> revolute
- joint right_ankle_x: type continuous -> fixed
- joint right_ankle_y: limit (none) -> lower=-0.7 upper=0.7 effort=100.0 velocity=10.0; type continuous -> revolute
- joint right_elbow: axis 0.00000 -1.00000 1.00000 -> 0.00000 1.00000 0.00000; limit (none) -> lower=0.0 upper=2.5 effort=100.0 velocity=10.0; type continuous -> revolute
- joint right_hip_x: limit (none) -> lower=-0.8 upper=0.8 effort=100.0 velocity=10.0; type fixed -> revolute
- joint right_hip_y: type continuous -> fixed
- joint right_hip_z: limit (none) -> lower=-1.5 upper=0.5 effort=100.0 velocity=10.0; type continuous -> revolute
- joint right_knee: limit (none) -> lower=0.0 upper=2.0 effort=100.0 velocity=10.0; type continuous -> revolute
- joint right_shoulder1: axis 2.00000 1.00000 1.00000 -> 0.00000 1.00000 0.00000; limit (none) -> lower=-2.0 upper=2.0 effort=100.0 velocity=10.0; type continuous -> revolute
- joint right_shoulder2: axis 0.00000 -1.00000 1.00000 -> 1.00000 0.00000 0.00000; limit (none) -> lower=-1.0 upper=1.0 effort=100.0 velocity=10.0; type continuous -> revolute

Commit message: look smroe liek human

File: data/humanoid.urdf (robot description, URDF)
Before this commit: robot , 34 links, 33 joints
Joints:
- joint abdomen_y: limit lower=-0.5 upper=0.5 effort=100.0 velocity=10.0 -> lower=-0.3 upper=0.7 effort=100.0 velocity=10.0
- joint abdomen_z: limit (none) -> lower=-0.5 upper=0.5 effort=100.0 velocity=10.0; type fixed -> revolute
- joint left_hip_x: limit lower=-0.8 upper=0.8 effort=100.0 velocity=10.0 -> lower=-1.0 upper=0.5 effort=100.0 velocity=10.0
- joint left_hip_y: limit (none) -> lower=-0.4 upper=2.0 effort=100.0 velocity=10.0; type fixed -> revolute
- joint left_hip_z: limit lower=-1.5 upper=0.5 effort=100.0 velocity=10.0 -> (none); type revolute -> fixed
- joint left_knee: axis 0.00000 -1.00000 0.00000 -> 0.00000 1.00000 0.00000; limit lower=0.0 upper=2.0 effort=100.0 velocity=10.0 -> lower=0.0 upper=2.5 effort=100.0 velocity=10.0
- joint right_hip_x: limit lower=-0.8 upper=0.8 effort=100.0 velocity=10.0 -> lower=-0.5 upper=1.0 effort=100.0 velocity=10.0
- joint right_hip_y: limit (none) -> lower=-0.4 upper=2.0 effort=100.0 velocity=10.0; type fixed -> revolute
- joint right_hip_z: limit lower=-1.5 upper=0.5 effort=100.0 velocity=10.0 -> (none); type revolute -> fixed
- joint right_knee: axis 0.00000 -1.00000 0.00000 -> 0.00000 1.00000 0.00000; limit lower=0.0 upper=2.0 effort=100.0 velocity=10.0 -> lower=0.0 upper=2.5 effort=100.0 velocity=10.0

Commit message: better humanoid motion

File: data/humanoid.urdf (robot description, URDF)
Before this commit: robot , 34 links, 33 joints
Joints:
- joint left_hip_y: limit lower=-0.4 upper=2.0 effort=100.0 velocity=10.0 -> lower=-2.0 upper=2.0 effort=100.0 velocity=10.0
- joint left_shoulder2: limit lower=-1.0 upper=1.0 effort=100.0 velocity=10.0 -> lower=-2.0 upper=2.0 effort=100.0 velocity=10.0
- joint right_hip_y: limit lower=-0.4 upper=2.0 effort=100.0 velocity=10.0 -> lower=-2.0 upper=2.0 effort=100.0 velocity=10.0
- joint right_shoulder2: limit lower=-1.0 upper=1.0 effort=100.0 velocity=10.0 -> lower=-2.0 upper=2.0 effort=100.0 velocity=10.0

Commit message: added joint controls

File: data/humanoid.urdf (robot description, URDF)
Before this commit: robot , 34 links, 33 joints
Links:
- removed link left_foot
- removed link left_lower_arm
- removed link left_shin
- removed link left_thigh
- removed link left_upper_arm
- removed link link1_11
- removed link link1_13
- removed link link1_14
- removed link link1_16
- removed link link1_17
- removed link link1_18
- removed link link1_2
- removed link link1_20
- removed link link1_22
- removed link link1_23
- removed link link1_25
- removed link link1_26
- removed link link1_28
- removed link link1_3
- removed link link1_30
- removed link link1_31
- removed link link1_33
- removed link link1_5
- removed link link1_7
- removed link link1_8
- removed link link1_9
- removed link lwaist
- removed link pelvis
- removed link right_foot
- removed link right_lower_arm
- removed link right_shin
- removed link right_thigh
- removed link right_upper_arm
- removed link torso
- added link left_foot_object, mass 1.13114; collision box size=0.05400 0.05400 0.21095
- added link left_lower_arm_object, mass 1.22954; collision box size=0.06200 0.06200 0.27713
- added link left_shin_object, mass 2.75570; collision box size=0.09800 0.09800 0.30000
- added link left_thigh_object, mass 4.75175; collision box size=0.12000 0.12000 0.34015
- added link left_upper_arm_object, mass 1.66108; collision box size=0.08000 0.08000 0.27713
- added link pelvis_object, mass 6.61619; collision box size=0.18000 0.18000 0.14000
- added link right_foot_object, mass 1.13114; collision box size=0.05400 0.05400 0.21095
- added link right_lower_arm_object, mass 1.22954; collision box size=0.06200 0.06200 0.27713
- added link right_shin_object, mass 2.75570; collision box size=0.09800 0.09800 0.30000
- added link right_thigh_object, mass 4.75175; collision box size=0.12000 0.12000 0.34015
- added link right_upper_arm_object, mass 1.66108; collision box size=0.08000 0.08000 0.27713
- added link torso_object, mass 8.90746; collision box size=0.14000 0.14000 0.14000
- added link waist_object, mass 2.26195; collision box size=0.12000 0.12000 0.12000
Joints:
- removed joint abdomen_x
- removed joint abdomen_y
- removed joint jointfix_0_14
- removed joint jointfix_10_33
- removed joint jointfix_11_31
- removed joint jointfix_1_11
- removed joint jointfix_2_9
- removed joint jointfix_3_23
- removed joint jointfix_4_20
- removed joint jointfix_5_18
- removed joint jointfix_6_5
- removed joint jointfix_7_3
- removed joint jointfix_8_28
- removed joint jointfix_9_26
- removed joint left_ankle_x
- removed joint left_hip_y
- removed joint left_hip_z
- removed joint left_shoulder2
- removed joint right_ankle_x
- removed joint right_hip_y
- removed joint right_hip_z
- removed joint right_shoulder2
- added joint waist_to_pelvis_y: type revolute, parent waist_object, child pelvis_object, origin xyz=0.00000 0.00000 -0.10000 rpy=0.00000 -0.00000 0.00000, axis 0.00000 1.00000 0.00000, limit lower=-0.3 upper=0.7 effort=100.0 velocity=10.0
- joint abdomen_z: child link1_2 -> waist_object; parent torso -> torso_object
- joint left_ankle_y: child link1_22 -> left_foot_object; parent left_shin -> left_shin_object
- joint left_elbow: child link1_33 -> left_lower_arm_object; parent left_upper_arm -> left_upper_arm_object
- joint left_hip_x: child link1_16 -> left_thigh_object; limit lower=-1.0 upper=0.5 effort=100.0 velocity=10.0 -> lower=-0.5 upper=1.0 effort=100.0 velocity=10.0; parent pelvis -> pelvis_object
- joint left_knee: child link1_20 -> left_shin_object; parent left_thigh -> left_thigh_object
- joint left_shoulder1: child link1_30 -> left_upper_arm_object; parent torso -> torso_object
- joint right_ankle_y: child link1_13 -> right_foot_object; parent right_shin -> right_shin_object
- joint right_elbow: child link1_28 -> right_lower_arm_object; parent right_upper_arm -> right_upper_arm_object
- joint right_hip_x: child link1_7 -> right_thigh_object; limit lower=-0.5 upper=1.0 effort=100.0 velocity=10.0 -> lower=-1.0 upper=0.5 effort=100.0 velocity=10.0; parent pelvis -> pelvis_object
- joint right_knee: child link1_11 -> right_shin_object; parent right_thigh -> right_thigh_object
- joint right_shoulder1: child link1_25 -> right_upper_arm_object; parent torso -> torso_object

Commit message: added key animation

File: data/humanoid.urdf (robot description, URDF)
Before this commit: robot humanoid_objects, 13 links, 12 joints
Links:
- added link head_object, mass 2.0; collision sphere radius=0.10
Joints:
- added joint neck_joint: type revolute, parent torso_object, child head_object, origin xyz=0.00000 0.00000 0.20000 rpy=0.00000 0.00000 0.00000, axis 0.00000 1.00000 0.00000, limit lower=-0.5 upper=0.5 effort=100.0 velocity=10.0

Commit message: added Env3D sub base class

File: data/humanoid.urdf (robot description, URDF)
Before this commit: robot humanoid_objects, 14 links, 13 joints
Joints:
- joint neck_joint: origin xyz=0.00000 0.00000 0.20000 rpy=0.00000 0.00000 0.00000 -> xyz=0.00000 0.00000 0.00000 rpy=0.00000 0.00000 0.00000

Commit message: Added a manipulator class for joints

File: data/humanoid.urdf (robot description, URDF)
Before this commit: robot humanoid_objects, 14 links, 13 joints
Joints:
- joint waist_to_pelvis_y: limit lower=-0.3 upper=0.7 effort=100.0 velocity=10.0 -> lower=-1.3 upper=0.7 effort=100.0 velocity=10.0

Commit message: fixed urdf files with shoulder and elbow controls

File: data/humanoid.urdf (robot description, URDF)
Before this commit: robot humanoid_objects, 14 links, 13 joints
Links:
- added link left_shoulder_flex_link, mass 0.001; collision sphere radius=0.001
- added link left_shoulder_out_link, mass 0.001; collision sphere radius=0.001
- added link right_shoulder_flex_link, mass 0.001; collision sphere radius=0.001
- added link right_shoulder_out_link, mass 0.001; collision sphere radius=0.001
Joints:
- removed joint left_elbow
- removed joint left_shoulder1
- removed joint right_elbow
- removed joint right_shoulder1
- added joint left_elbow_flex: type revolute, parent left_upper_arm_object, child left_lower_arm_object, origin xyz=0.18000 0.18000 -0.18000 rpy=0.00000 -0.00000 0.00000, axis 0.00000 -1.00000 -1.00000, limit lower=-2.0 upper=1.0 effort=100.0 velocity=10.0
- added joint left_shoulder_flex: type revolute, parent torso_object, child left_shoulder_flex_link, origin xyz=0.00000 0.17000 0.06000 rpy=0.00000 -0.00000 0.00000, axis 0.00000 1.00000 0.00000, limit lower=-2.0 upper=2.0 effort=100.0 velocity=10.0
- added joint left_shoulder_out: type revolute, parent left_shoulder_flex_link, child left_shoulder_out_link, origin xyz=0.00000 0.00000 0.00000 rpy=0.00000 0.00000 0.00000, axis -1.00000 0.00000 0.00000, limit lower=-1.5 upper=1.5 effort=100.0 velocity=10.0
- added joint left_shoulder_rotate: type revolute, parent left_shoulder_out_link, child left_upper_arm_object, origin xyz=0.00000 0.00000 0.00000 rpy=0.00000 0.00000 0.00000, axis 0.00000 0.00000 -1.00000, limit lower=-1.5 upper=1.5 effort=100.0 velocity=10.0
- added joint right_elbow_flex: type revolute, parent right_upper_arm_object, child right_lower_arm_object, origin xyz=0.18000 -0.18000 -0.18000 rpy=0.00000 -0.00000 0.00000, axis 0.00000 -1.00000 1.00000, limit lower=-2.0 upper=1.0 effort=100.0 velocity=10.0
- added joint right_shoulder_flex: type revolute, parent torso_object, child right_shoulder_flex_link, origin xyz=0.00000 -0.17000 0.06000 rpy=0.00000 -0.00000 0.00000, axis 0.00000 1.00000 0.00000, limit lower=-2.0 upper=2.0 effort=100.0 velocity=10.0
- added joint right_shoulder_out: type revolute, parent right_shoulder_flex_link, child right_shoulder_out_link, origin xyz=0.00000 0.00000 0.00000 rpy=0.00000 0.00000 0.00000, axis 1.00000 0.00000 0.00000, limit lower=-1.5 upper=1.5 effort=100.0 velocity=10.0
- added joint right_shoulder_rotate: type revolute, parent right_shoulder_out_link, child right_upper_arm_object, origin xyz=0.00000 0.00000 0.00000 rpy=0.00000 0.00000 0.00000, axis 0.00000 0.00000 1.00000, limit lower=-1.5 upper=1.5 effort=100.0 velocity=10.0

Commit message: clean up

File: data/humanoid.urdf (robot description, URDF)
Before this commit: robot humanoid_objects, 18 links, 17 joints
Links:
- added link left_hip_link, mass 0.001; collision sphere radius=0.001
- added link right_hip_link, mass 0.001; collision sphere radius=0.001
Joints:
- added joint left_hip_y: type revolute, parent left_hip_link, child left_thigh_object, origin xyz=0.00000 0.00000 0.00000 rpy=0.00000 -0.00000 0.00000, axis 0.00000 1.00000 0.00000, limit lower=-2.5 upper=1.5 effort=100.0 velocity=10.0
- added joint right_hip_y: type revolute, parent right_hip_link, child right_thigh_object, origin xyz=0.00000 0.00000 0.00000 rpy=0.00000 -0.00000 0.00000, axis 0.00000 1.00000 0.00000, limit lower=-2.5 upper=1.5 effort=100.0 velocity=10.0
- joint left_hip_x: child left_thigh_object -> left_hip_link
- joint right_hip_x: child right_thigh_object -> right_hip_link
