Commit message: removed grid and grid spacing

File: data/humanstand.urdf (robot description, URDF)
Before this commit: robot humanoid_objects, 14 links, 13 joints
Links:
- removed link pelvis_object
- removed link waist_object
- added link left_butt_object, mass 3.308095; collision box size=0.09000 0.08000 0.14000
- added link right_butt_object, mass 3.308095; collision box size=0.09000 0.08000 0.14000
Joints:
- removed joint abdomen_z
- removed joint waist_to_pelvis_y
- added joint torso_to_left_pelvis_y: type revolute, parent torso_object, child left_butt_object, origin xyz=-0.01026 0.07000 -0.25000 rpy=0.00000 -0.00000 0.00000, axis 0.00000 1.00000 0.00000, limit lower=-1.3 upper=0.7 effort=1000.0 velocity=1.0
- added joint torso_to_right_pelvis_y: type revolute, parent torso_object, child right_butt_object, origin xyz=-0.01026 -0.07000 -0.25000 rpy=0.00000 -0.00000 0.00000, axis 0.00000 1.00000 0.00000, limit lower=-1.3 upper=0.7 effort=1000.0 velocity=1.0
- joint left_ankle_y: limit lower=-0.7 upper=0.7 effort=100.0 velocity=10.0 -> lower=-0.7 upper=0.7 effort=1000.0 velocity=1.0
- joint left_elbow: limit lower=0.0 upper=2.5 effort=100.0 velocity=10.0 -> lower=0.0 upper=2.5 effort=1000.0 velocity=1.0
- joint left_hip_x: limit lower=-0.5 upper=1.0 effort=100.0 velocity=10.0 -> lower=-0.5 upper=1.0 effort=1000.0 velocity=1.0; origin xyz=0.00000 0.10000 -0.04000 rpy=0.00000 -0.00000 0.00000 -> xyz=0.02000 0.05500 -0.08000 rpy=0.00000 -0.00000 0.00000; parent pelvis_object -> left_butt_object
- joint left_knee: limit lower=0.0 upper=2.5 effort=100.0 velocity=10.0 -> lower=0.0 upper=2.5 effort=1000.0 velocity=1.0
- joint left_shoulder1: limit lower=-2.0 upper=2.0 effort=100.0 velocity=10.0 -> lower=-2.0 upper=2.0 effort=1000.0 velocity=1.0
- joint neck_joint: limit lower=-0.5 upper=0.5 effort=100.0 velocity=10.0 -> lower=-0.5 upper=0.5 effort=1000.0 velocity=1.0
- joint right_ankle_y: limit lower=-0.7 upper=0.7 effort=100.0 velocity=10.0 -> lower=-0.7 upper=0.7 effort=1000.0 velocity=1.0
- joint right_elbow: limit lower=0.0 upper=2.5 effort=100.0 velocity=10.0 -> lower=0.0 upper=2.5 effort=1000.0 velocity=1.0
- joint right_hip_x: limit lower=-1.0 upper=0.5 effort=100.0 velocity=10.0 -> lower=-1.0 upper=0.5 effort=1000.0 velocity=1.0; origin xyz=0.00000 -0.10000 -0.04000 rpy=0.00000 -0.00000 0.00000 -> xyz=0.02000 -0.05500 -0.04000 rpy=0.00000 -0.00000 0.00000; parent pelvis_object -> right_butt_object
- joint right_knee: limit lower=0.0 upper=2.5 effort=100.0 velocity=10.0 -> lower=0.0 upper=2.5 effort=1000.0 velocity=1.0
- joint right_shoulder1: limit lower=-2.0 upper=2.0 effort=100.0 velocity=10.0 -> lower=-2.0 upper=2.0 effort=1000.0 velocity=1.0
