Commit message: increase plane size, update env

File: data/goat.urdf (robot description, URDF)
Before this commit: robot four_legged_creature, 6 links, 5 joints
Links:
- removed link front_left_leg_object
- removed link front_right_leg_object
- removed link rear_left_leg_object
- removed link rear_right_leg_object
- added link front_left_leg_lower_object, mass 2.37588; collision box size=0.08000 0.08000 0.64015
- added link front_left_leg_upper_object, mass 2.37588; collision box size=0.08000 0.64015 0.08000
- added link front_right_leg_lower_object, mass 2.37588; collision box size=0.08000 0.08000 0.64015
- added link front_right_leg_upper_object, mass 2.37588; collision box size=0.64015 0.08000 0.08000
- added link rear_left_leg_lower_object, mass 2.37588; collision box size=0.08000 0.08000 0.64015
- added link rear_left_leg_upper_object, mass 2.37588; collision box size=0.64015 0.08000 0.08000
- added link rear_right_leg_lower_object, mass 2.37588; collision box size=0.08000 0.08000 0.64015
- added link rear_right_leg_upper_object, mass 2.37588; collision box size=0.08000 0.64015 0.08000
Joints:
- removed joint torso_to_front_left_leg
- removed joint torso_to_front_right_leg
- removed joint torso_to_rear_left_leg
- removed joint torso_to_rear_right_leg
- added joint front_left_leg_upper_to_lower: type revolute, parent front_left_leg_upper_object, child front_left_leg_lower_object, origin xyz=0.00000 0.64015 0.00000 rpy=0 0 0, axis 1 0 0, limit lower=-0.5 upper=0.5 effort=1000.0 velocity=1.0
- added joint front_right_leg_upper_to_lower: type revolute, parent front_right_leg_upper_object, child front_right_leg_lower_object, origin xyz=0.64015 0.00000 0.00000 rpy=0 0 0, axis 0 1 0, limit lower=-0.5 upper=0.5 effort=1000.0 velocity=1.0
- added joint rear_left_leg_upper_to_lower: type revolute, parent rear_left_leg_upper_object, child rear_left_leg_lower_object, origin xyz=-0.64015 0.00000 0.00000 rpy=0 0 0, axis 0 1 0, limit lower=-0.5 upper=0.5 effort=1000.0 velocity=1.0
- added joint rear_right_leg_upper_to_lower: type revolute, parent rear_right_leg_upper_object, child rear_right_leg_lower_object, origin xyz=0.00000 -0.64015 0.00000 rpy=0 0 0, axis 1 0 0, limit lower=-0.5 upper=0.5 effort=1000.0 velocity=1.0
- added joint torso_to_front_left_leg_upper: type revolute, parent torso_object, child front_left_leg_upper_object, origin xyz=0.07000 0.07000 -0.07000 rpy=0.00000 0.00000 -1, axis 0 0 1, limit lower=-0.6 upper=0.6 effort=1000.0 velocity=1.0
- added joint torso_to_front_right_leg_upper: type revolute, parent torso_object, child front_right_leg_upper_object, origin xyz=0.07000 -0.07000 -0.07000 rpy=0.00000 0.00000 -1, axis 0 0 1, limit lower=-0.6 upper=0.6 effort=1000.0 velocity=1.0
- added joint torso_to_rear_left_leg_upper: type revolute, parent torso_object, child rear_left_leg_upper_object, origin xyz=-0.07000 0.07000 -0.07000 rpy=0.00000 0.00000 5.5, axis 0 0 1, limit lower=-0.6 upper=0.6 effort=1000.0 velocity=1.0
- added joint torso_to_rear_right_leg_upper: type revolute, parent torso_object, child rear_right_leg_upper_object, origin xyz=-0.07000 -0.07000 -0.07000 rpy=0.00000 0.00000 -1, axis 0 0 1, limit lower=-0.6 upper=0.6 effort=1000.0 velocity=1.0

File: data/plane.urdf (robot description, URDF)
Before this commit: robot plane, 1 links, 0 joints
Links:
- link planeLink: geometry collision box size=70 70 10; visual mesh filename=plane.obj scale=1 1 1
